File: rp2040/rp2040.kicad_sch (KiCad schematic)
At the start: 1 part, among them U1 RP2040

Commit message: .
Parts:
- added C1, C10, C15, C2, C3, C4, C5, C6, C7, C9: 100nF, Capacitor_SMD:C_0603_1608Metric, symbol Device:C_Small
- added C11, C12: 10uF, Capacitor_SMD:C_0603_1608Metric, symbol Device:C_Small
- added C13, C14: 27pF, Capacitor_SMD:C_0603_1608Metric, symbol Device:C_Small
- added C8: 1uF, Capacitor_SMD:C_0603_1608Metric, symbol Device:C_Small
- added J1: USB_B_Micro, Connector_USB:USB_Micro-B_GCT_USB3076-30-A, symbol Connector:USB_B_Micro
- added J2: Conn_01x02, symbol Connector_Generic:Conn_01x02
- added R1, R2: 27.4R, symbol Device:R_Small
- added R3: 10K, symbol Device:R_Small
- added R4: 1K, symbol Device:R_Small
- added U2: AMS1117-3.3, Package_TO_SOT_SMD:SOT-223-3_TabPin2, symbol Regulator_Linear:AMS1117-3.3
- added U3: W25Q128JVS, Package_SO:SOIC-8_5.23x5.23mm_P1.27mm, symbol Memory_Flash:W25Q128JVS
- added Y1: 12MHz, symbol Device:Crystal_Small
Connections:
- net +3.3V: now reaches U1.1 (IOVDD), U1.10 (IOVDD), U1.22 (IOVDD), U1.33 (IOVDD), U1.42 (IOVDD), U1.49 (IOVDD)
- net +3.3V: now also U1.43 (ADC_AVDD), U1.44 (VREG_IN), U1.48 (USB_VDD), C1.1, C12.1, C15.1, C2.1, C3.1, C4.1, C5.1, C6.1, C7.1, C8.1, R3.2, U2.2 (VO), U3.8 (VCC)
- net GPIO8: now reaches U1.11 (GPIO8)
- net GPIO9: now reaches U1.12 (GPIO9)
- net GPIO10: now reaches U1.13 (GPIO10)
- net GPIO11: now reaches U1.14 (GPIO11)
- net GPIO12: now reaches U1.15 (GPIO12)
- net GPIO13: now reaches U1.16 (GPIO13)
- net GPIO14: now reaches U1.17 (GPIO14)
- net GPIO15: now reaches U1.18 (GPIO15)
- net TESTEN: now reaches U1.19 (TESTEN)
- net GPIO0: now reaches U1.2 (GPIO0)
- net XIN: now reaches U1.20 (XIN)
- net XIN: now also C13.2, Y1.2
- net XOUT: now reaches U1.21 (XOUT)
- net XOUT: now also C14.2, Y1.1
- net +1V1: now reaches U1.23 (DVDD), U1.50 (DVDD)
- net +1V1: now also U1.45 (VREG_VOUT), U1.57 (GND), C10.1, C10.2, C11.2, C12.2, C13.1, C14.1, C15.2, C8.2, C9.1, C9.2, J1.5 (GND), J1.6 (Shield), J2.1 (Pin_1), U2.1 (GND), U3.4 (GND)
- net SWCLK: now reaches U1.24 (SWCLK)
- net SWD: now reaches U1.25 (SWD)
- net GPIO16: now reaches U1.27 (GPIO16)
- net GPIO17: now reaches U1.28 (GPIO17)
- net GPIO18: now reaches U1.29 (GPIO18)
- net GPIO1: now reaches U1.3 (GPIO1)
- net GPIO19: now reaches U1.30 (GPIO19)
- net GPIO20: now reaches U1.31 (GPIO20)
- net GPIO21: now reaches U1.32 (GPIO21)
- net GPIO22: now reaches U1.34 (GPIO22)
- net GPIO23: now reaches U1.35 (GPIO23)
- net GPIO24: now reaches U1.36 (GPIO24)
- net GPIO25: now reaches U1.37 (GPIO25)
- net GPIO26_ADC0: now reaches U1.38 (GPIO26_ADC0)
- net GPIO27_ADC1: now reaches U1.39 (GPIO27_ADC1)
- net GPIO2: now reaches U1.4 (GPIO2)
- net GPIO28_ADC2: now reaches U1.40 (GPIO28_ADC2)
- net GPIO29_ADC3: now reaches U1.41 (GPIO29_ADC3)
- net at U1.46 (USB_DM): now also R2.2
- net at U1.47 (USB_DP): now also R1.2
- net GPIO3: now reaches U1.5 (GPIO3)
- net QSPI_SD3: now reaches U1.51 (QSPI_SD3)
- net QSPI_SD3: now also U3.7 (IO3)
- net QSPI_SCLK: now reaches U1.52 (QSPI_SCLK)
- net QSPI_SCLK: now also U3.6 (CLK)
- net QSPI_SD0: now reaches U1.53 (QSPI_SD0)
- net QSPI_SD0: now also U3.5 (DI(IO0))
- net QSPI_SD2: now reaches U1.54 (QSPI_SD2)
- net QSPI_SD2: now also U3.3 (IO2)
- net QSPI_SD1: now reaches U1.55 (QSPI_SD1)
- net QSPI_SD1: now also U3.2 (DO(IO1))
- net QSPI_SS: now reaches U1.56 (QSPI_SS)
- net QSPI_SS: now also R3.1, R4.1, U3.1 (~{CS})
- net GPIO4: now reaches U1.6 (GPIO4)
- net GPIO5: now reaches U1.7 (GPIO5)
- net GPIO6: now reaches U1.8 (GPIO6)
- net GPIO7: now reaches U1.9 (GPIO7)
- new net: C11.1, J1.1 (VBUS), U2.3 (VI)
- new net: C1.2, C2.2, C3.2, C4.2, C5.2, C6.2, C7.2
- new net: J2.2 (Pin_2), R4.2
- new net USB_D+: J1.3 (D+), R1.1
- new net USB_D-: J1.2 (D-), R2.1
- no-connect marks 0 -> 1
Other:
- moved on the sheet: U1

Commit message: .
Parts:
- removed J2: Conn_01x02, symbol Connector_Generic:Conn_01x02
- removed Y1: 12MHz, symbol Device:Crystal_Small
- added C1: 100nF, Capacitor_SMD:C_0805_2012Metric, symbol Device:C_Small
- added C2: 1uF, Capacitor_SMD:C_0603_1608Metric, symbol Device:C_Small
- added D1, D2: LED_ORANGE, LED_SMD:LED_0805_2012Metric, symbol Device:LED_Small
- added H? (x4): MountingHole, MountingHole:MountingHole_2.7mm_M2.5, symbol Mechanical:MountingHole
- added J2, J4: Conn_01x18, Connector_PinHeader_2.54mm:PinHeader_1x18_P2.54mm_Vertical, symbol Connector_Generic:Conn_01x18
- added J3: Conn_01x02, Connector_PinHeader_2.54mm:PinHeader_1x02_P2.54mm_Vertical, symbol Connector_Generic:Conn_01x02
- added Q1, Q2: 2N7002, Package_TO_SOT_SMD:SOT-23, symbol Transistor_FET:2N7002
- added R11: 1K, Resistor_SMD:R_0603_1608Metric, symbol Device:R_Small
- added R3, R4: 4K7, Resistor_SMD:R_0805_2012Metric, symbol Device:R_Small_US
- added R5, R8: 10K, Resistor_SMD:R_0805_2012Metric, symbol Device:R_Small_US
- added R6, R9: 330R, Resistor_SMD:R_0805_2012Metric, symbol Device:R_Small_US
- added SW1: 6x6_SMD_BUTTON, Button_Switch_SMD:SW_SPST_CK_RS282G05A3, symbol Switch:SW_Push
- added U1: AT24C02C, Package_SO:SOIC-8_3.9x4.9mm_P1.27mm, symbol Memory_EEPROM:M24C01-WMN
- added U5: SSD1306_CRY, GOFootprint:128x64OLED, symbol GOSymbol:SSD1306_CRY
- added Y?: 12MHz, Crystal:Crystal_SMD_5032-4Pin_5.0x3.2mm, symbol Device:Crystal_GND24_Small
- R1, R2: footprint (none) -> Resistor_SMD:R_0603_1608Metric
- R10: renamed from R3; footprint (none) -> Resistor_SMD:R_0603_1608Metric
- R7: renamed from R4; footprint (none) -> Resistor_SMD:R_0603_1608Metric
- renumbered C6 to C10, C7 to C11, C8 to C12, C11 to C15, C15 to C16, C12 to C17, C10 to C3, C9 to C4, C1 to C5, C2 to C6, C3 to C7, C4 to C8, C5 to C9, U1 to U2, U2 to U4
Connections:
- net +1V1: now also C2.1; no longer C12.2, C13.1, C14.1, C15.2, C16.2, C17.2, C3.2, C4.2, J1.5 (GND), J1.6 (Shield), U2.57 (GND), U3.4 (GND), U4.1 (GND)
- net +3.3V: now also C1.2, J2.1 (Pin_1), J3.2 (Pin_2), R3.1, R4.1, R6.2, R9.2, U1.8 (VCC)
- net GPIO0: now also J2.2 (Pin_2), U5.4 (SDA)
- net GPIO1: now also J2.3 (Pin_3), U5.3 (SCL)
- net GPIO10: now also J2.12 (Pin_12)
- net GPIO11: now also J2.13 (Pin_13)
- net GPIO12: now also J2.14 (Pin_14)
- net GPIO13: now also J2.15 (Pin_15)
- net GPIO14: now also J2.16 (Pin_16), Q1.1 (G), R5.1
- net GPIO15: now also J2.17 (Pin_17), Q2.1 (G), R8.1
- net GPIO16: now also J4.14 (Pin_14)
- net GPIO17: now also J4.13 (Pin_13)
- net GPIO18: now also J4.12 (Pin_12)
- net GPIO19: now also J4.11 (Pin_11)
- net GPIO2: now also J2.4 (Pin_4), R3.2, U1.5 (SDA)
- net GPIO20: now also J4.10 (Pin_10)
- net GPIO21: now also J4.9 (Pin_9)
- net GPIO22: now also J4.8 (Pin_8)
- net GPIO23: now also J4.7 (Pin_7)
- net GPIO24: now also J4.6 (Pin_6)
- net GPIO25: now also J4.5 (Pin_5)
- net GPIO26_ADC0: now also J4.4 (Pin_4)
- net GPIO27_ADC1: now also J4.3 (Pin_3)
- net GPIO28_ADC2: now also J4.2 (Pin_2)
- net GPIO29_ADC3: now also J4.1 (Pin_1)
- net GPIO3: now also J2.5 (Pin_5), R4.2, U1.6 (SCL)
- net GPIO4: now also J2.6 (Pin_6)
- net GPIO5: now also J2.7 (Pin_7)
- net GPIO6: now also J2.8 (Pin_8)
- net GPIO7: now also J2.9 (Pin_9)
- net GPIO8: now also J2.10 (Pin_10)
- net GPIO9: now also J2.11 (Pin_11)
- net SWCLK: now also J4.17 (Pin_17)
- net SWD: now also J4.16 (Pin_16)
- net XIN: now also Y?.3
- net XOUT: now also R11.1; no longer C14.2
- net at R7.2: now also SW1.2
- net RUN: now reaches U2.26 (RUN)
- net RUN: now also J4.15 (Pin_15)
- net TESTEN renamed GND
- net GND: now also C12.2, C13.1, C14.1, C15.2, C16.2, C17.2, C3.2, C4.2, J1.5 (GND), J1.6 (Shield), U2.57 (GND), U3.4 (GND), U4.1 (GND), C1.1, C2.2, J2.18 (Pin_18), J4.18 (Pin_18), Q1.2 (S), Q2.2 (S), R5.2, R8.2, SW1.1, U1.1 (E0), U1.2 (E1), U1.3 (E2), U1.4 (VSS), U1.7 (~{WC}), U5.2 (GND), Y?.2, Y?.4
- new net: D2.1 (K), Q2.3 (D)
- new net: C14.2, R11.2, Y?.1
- new net: D1.1 (K), Q1.3 (D)
- new net: D2.2 (A), R9.1
- new net: D1.2 (A), R6.1
- new net: J3.1 (Pin_1), U5.1 (VCC)

Commit message: .
Parts:
- removed H? (x4): MountingHole, MountingHole:MountingHole_2.7mm_M2.5, symbol Mechanical:MountingHole
Changed lines of the file:
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@@
-    )
-  )
-  (symbol (lib_id "Mechanical:MountingHole") (at 265.43 15.24 0) (unit 1)
-    (in_bom yes) (on_board yes) (dnp no)
-    (property "Reference" "H?" (at 267.97 14.0716 0)
-      (effects (font (size 1.27 1.27)) (justify left))
-    )
-    (property "Value" "MountingHole" (at 267.97 16.383 0)
-      (effects (font (size 1.27 1.27)) (justify left))
-    )
-    (property "Footprint" "MountingHole:MountingHole_2.7mm_M2.5" (at 265.43 15.24 0)
-      (effects (font (size 1.27 1.27)) hide)
-    )
-    (property "Datasheet" "~" (at 265.43 15.24 0)
-      (effects (font (size 1.27 1.27)) hide)
-    )
-    (instances
-      (project "RP2040_minimal"
-        (path "/916eaa38-3a53-4e97-83dc-c40e06d8967b"
-          (reference "H?") (unit 1)
-        )
-      )
-      (project "rp2040"
-        (path "/c9598c3f-0f3a-4c4d-ac85-07132829eac5"
-          (reference "H1") (unit 1)
-        )
-      )
     )
   )
@@
         (path "/c9598c3f-0f3a-4c4d-ac85-07132829eac5"
           (reference "#PWR016") (unit 1)
-        )
-      )
-    )
-  )
-  (symbol (lib_id "Mechanical:MountingHole") (at 265.43 20.32 0) (unit 1)
-    (in_bom yes) (on_board yes) (dnp no)
-    (property "Reference" "H?" (at 267.97 19.1516 0)
-      (effects (font (size 1.27 1.27)) (justify left))
-    )
-    (property "Value" "MountingHole" (at 267.97 21.463 0)
-      (effects (font (size 1.27 1.27)) (justify left))
-    )
-    (property "Footprint" "MountingHole:MountingHole_2.7mm_M2.5" (at 265.43 20.32 0)
-      (effects (font (size 1.27 1.27)) hide)
-    )
-    (property "Datasheet" "~" (at 265.43 20.32 0)
-      (effects (font (size 1.27 1.27)) hide)
-    )
-    (instances
-      (project "RP2040_minimal"
-        (path "/916eaa38-3a53-4e97-83dc-c40e06d8967b"
-          (reference "H?") (unit 1)
-        )
-      )
-      (project "rp2040"
-        (path "/c9598c3f-0f3a-4c4d-ac85-07132829eac5"
-          (reference "H2") (unit 1)
         )
       )
@@
     )
   )
-  (symbol (lib_id "Mechanical:MountingHole") (at 265.43 25.4 0) (unit 1)
-    (in_bom yes) (on_board yes) (dnp no)
-    (property "Reference" "H?" (at 267.97 24.2316 0)
-      (effects (font (size 1.27 1.27)) (justify left))
-    )
-    (property "Value" "MountingHole" (at 267.97 26.543 0)
-      (effects (font (size 1.27 1.27)) (justify left))
-    )
-    (property "Footprint" "MountingHole:MountingHole_2.7mm_M2.5" (at 265.43 25.4 0)
-      (effects (font (size 1.27 1.27)) hide)
-    )
-    (property "Datasheet" "~" (at 265.43 25.4 0)
-      (effects (font (size 1.27 1.27)) hide)
-    )
-    (instances
-      (project "RP2040_minimal"
-        (path "/916eaa38-3a53-4e97-83dc-c40e06d8967b"
-          (reference "H?") (unit 1)
-        )
-      )
-      (project "rp2040"
-        (path "/c9598c3f-0f3a-4c4d-ac85-07132829eac5"
-          (reference "H3") (unit 1)
-        )
-      )
-    )
-  )
   (symbol (lib_id "Device:R_Small_US") (at 157.48 161.29 180) (unit 1)
     (in_bom yes) (on_board yes) (dnp no) (fields_autoplaced)
@@
         )
       )
-    )
-  )
-  (symbol (lib_id "Mechanical:MountingHole") (at 265.43 30.48 0) (unit 1)
-    (in_bom yes) (on_board yes) (dnp no)
-    (property "Reference" "H?" (at 267.97 29.3116 0)
-      (effects (font (size 1.27 1.27)) (justify left))
-    )
-    (property "Value" "MountingHole" (at 267.97 31.623 0)
-      (effects (font (size 1.27 1.27)) (justify left))
-    )
-    (property "Footprint" "MountingHole:MountingHole_2.7mm_M2.5" (at 265.43 30.48 0)
-      (effects (font (size 1.27 1.27)) hide)
-    )
-    (property "Datasheet" "~" (at 265.43 30.48 0)
-      (effects (font (size 1.27 1.27)) hide)
-    )
-    (instances
-      (project "RP2040_minimal"
-        (path "/916eaa38-3a53-4e97-83dc-c40e06d8967b"
-          (reference "H?") (unit 1)
-        )
-      )
-      (project "rp2040"
-        (path "/c9598c3f-0f3a-4c4d-ac85-07132829eac5"
-          (reference "H4") (unit 1)
-        )
-      )

Commit message: edit pcb
Parts:
- added H1, H2, H3, H4: MountingHole, MountingHole:MountingHole_3.2mm_M3_Pad_Via, symbol Mechanical:MountingHole
Connections:
- net GND: now also C10.2, C11.2, C5.2, C6.2, C7.2, C8.2, C9.2
- net VBUS: now reaches C15.1, J1.1 (VBUS), U4.3 (VI)
Changed lines of the file:
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@@
   (junction (at 162.56 129.54) (diameter 0) (color 0 0 0 0)
   )
+  (junction (at 118.11 43.18) (diameter 0) (color 0 0 0 0)
+  )
   (junction (at 83.82 35.56) (diameter 0) (color 0 0 0 0)
   )
@@
   )
   (junction (at 92.71 34.29) (diameter 0) (color 0 0 0 0)
+  )
+  (junction (at 118.11 34.29) (diameter 0) (color 0 0 0 0)
   )
   (junction (at 158.75 129.54) (diameter 0) (color 0 0 0 0)
@@
     (stroke (width 0) (type default))
   )
+  (wire (pts (xy 121.92 34.29) (xy 121.92 43.18))
+    (stroke (width 0) (type default))
+  )
   (wire (pts (xy 234.95 106.68) (xy 237.49 106.68))
     (stroke (width 0) (type default))
@@
     (stroke (width 0) (type default))
   )
+  (wire (pts (xy 118.11 34.29) (xy 121.92 34.29))
+    (stroke (width 0) (type default))
+  )
   (wire (pts (xy 240.03 49.53) (xy 240.03 52.07))
     (stroke (width 0) (type default))
@@
     (stroke (width 0) (type default))
   )
+  (wire (pts (xy 118.11 43.18) (xy 121.92 43.18))
+    (stroke (width 0) (type default))
+  )
   (wire (pts (xy 68.58 26.67) (xy 68.58 35.56))
     (stroke (width 0) (type default))
@@
     (effects (font (size 1.27 1.27)) (justify left))
     (property "Intersheetrefs" "${INTERSHEET_REFS}" (at 246.0806 101.6 0)
+      (effects (font (size 1.27 1.27)) (justify left) hide)
+    )
+  )
+  (global_label "VBUS" (shape input) (at 165.1 48.26 90) (fields_autoplaced)
+    (effects (font (size 1.27 1.27)) (justify left))
+    (property "Intersheetrefs" "${INTERSHEET_REFS}" (at 165.1 40.4556 90)
       (effects (font (size 1.27 1.27)) (justify left) hide)
     )
@@
     )
   )
+  (symbol (lib_id "Mechanical:MountingHole") (at 260.35 149.86 0) (unit 1)
+    (in_bom yes) (on_board yes) (dnp no) (fields_autoplaced)
+    (property "Reference" "H1" (at 262.89 149.225 0)
+      (effects (font (size 1.27 1.27)) (justify left))
+    )
+    (property "Value" "MountingHole" (at 262.89 151.765 0)
+      (effects (font (size 1.27 1.27)) (justify left))
+    )
+    (property "Footprint" "MountingHole:MountingHole_3.2mm_M3_Pad_Via" (at 260.35 149.86 0)
+      (effects (font (size 1.27 1.27)) hide)
+    )
+    (property "Datasheet" "~" (at 260.35 149.86 0)
+      (effects (font (size 1.27 1.27)) hide)
+    )
+    (instances
+      (project "rp2040"
+        (path "/c9598c3f-0f3a-4c4d-ac85-07132829eac5"
+          (reference "H1") (unit 1)
+        )
+      )
+    )
+  )
   (symbol (lib_id "power:GND") (at 158.75 90.17 270) (unit 1)
     (in_bom yes) (on_board yes) (dnp no)
@@
         (path "/c9598c3f-0f3a-4c4d-ac85-07132829eac5"
           (reference "#PWR025") (unit 1)
+        )
+      )
+    )
+  )
+  (symbol (lib_id "Mechanical:MountingHole") (at 245.5618 149.9 0) (unit 1)
+    (in_bom yes) (on_board yes) (dnp no) (fields_autoplaced)
+    (property "Reference" "H4" (at 248.1018 149.265 0)
+      (effects (font (size 1.27 1.27)) (justify left))
+    )
+    (property "Value" "MountingHole" (at 248.1018 151.805 0)
+      (effects (font (size 1.27 1.27)) (justify left))
+    )
+    (property "Footprint" "MountingHole:MountingHole_3.2mm_M3_Pad_Via" (at 245.5618 149.9 0)
+      (effects (font (size 1.27 1.27)) hide)
+    )
+    (property "Datasheet" "~" (at 245.5618 149.9 0)
+      (effects (font (size 1.27 1.27)) hide)
+    )
+    (instances
+      (project "rp2040"
+        (path "/c9598c3f-0f3a-4c4d-ac85-07132829eac5"
+          (reference "H4") (unit 1)
         )
       )
@@
     )
   )
+  (symbol (lib_id "Mechanical:MountingHole") (at 245.6985 156.3229 0) (unit 1)
+    (in_bom yes) (on_board yes) (dnp no) (fields_autoplaced)
+    (property "Reference" "H3" (at 248.2385 155.6879 0)
+      (effects (font (size 1.27 1.27)) (justify left))
+    )
+    (property "Value" "MountingHole" (at 248.2385 158.2279 0)
+      (effects (font (size 1.27 1.27)) (justify left))
+    )
+    (property "Footprint" "MountingHole:MountingHole_3.2mm_M3_Pad_Via" (at 245.6985 156.3229 0)
+      (effects (font (size 1.27 1.27)) hide)
+    )
+    (property "Datasheet" "~" (at 245.6985 156.3229 0)
+      (effects (font (size 1.27 1.27)) hide)
+    )
+    (instances
+      (project "rp2040"
+        (path "/c9598c3f-0f3a-4c4d-ac85-07132829eac5"
+          (reference "H3") (unit 1)
+        )
+      )
+    )
+  )
   (symbol (lib_id "Device:C_Small") (at 195.58 54.61 0) (unit 1)
     (in_bom yes) (on_board yes) (dnp no)
@@
         )
       )
+    )
+  )
+  (symbol (lib_id "Mechanical:MountingHole") (at 260.3208 157.4162 0) (unit 1)
+    (in_bom yes) (on_board yes) (dnp no) (fields_autoplaced)
+    (property "Reference" "H2" (at 262.8608 156.7812 0)
+      (effects (font (size 1.27 1.27)) (justify left))
+    )
+    (property "Value" "MountingHole" (at 262.8608 159.3212 0)
+      (effects (font (size 1.27 1.27)) (justify left))
+    )
+    (property "Footprint" "MountingHole:MountingHole_3.2mm_M3_Pad_Via" (at 260.3208 157.4162 0)
+      (effects (font (size 1.27 1.27)) hide)
+    )
+    (property "Datasheet" "~" (at 260.3208 157.4162 0)
+      (effects (font (size 1.27 1.27)) hide)
+    )
+    (instances
+      (project "rp2040"
+        (path "/c9598c3f-0f3a-4c4d-ac85-07132829eac5"
+          (reference "H2") (unit 1)
+        )
+      )

Commit message: add Reset buton
Parts:
- added R12: 1K, Resistor_SMD:R_0805_2012Metric, symbol Device:R_Small_US
- added SW2: 6x6_SMD_BUTTON, Button_Switch_SMD:SW_SPST_CK_RS282G05A3, symbol Switch:SW_Push
Connections:
- net +3.3V: now also R12.2
- net GND: now also SW2.1
- net RUN: now also R12.1, SW2.2
Changed lines of the file:
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@@
   (junction (at 92.71 34.29) (diameter 0) (color 0 0 0 0)
   )
+  (junction (at 46.99 46.99) (diameter 0) (color 0 0 0 0)
+  )
   (junction (at 118.11 34.29) (diameter 0) (color 0 0 0 0)
   )
@@
     (stroke (width 0) (type default))
   )
+  (wire (pts (xy 46.99 41.91) (xy 46.99 46.99))
+    (stroke (width 0) (type default))
+  )
   (wire (pts (xy 64.77 186.69) (xy 64.77 179.07))
     (stroke (width 0) (type default))
@@
     (stroke (width 0) (type default))
   )
+  (wire (pts (xy 46.99 46.99) (xy 48.26 46.99))
+    (stroke (width 0) (type default))
+  )
   (wire (pts (xy 154.94 55.88) (xy 158.75 55.88))
     (stroke (width 0) (type default))
@@
     (stroke (width 0) (type default))
   )
-  (wire (pts (xy 45.72 46.99) (xy 48.26 46.99))
+  (wire (pts (xy 43.18 46.99) (xy 46.99 46.99))
     (stroke (width 0) (type default))
   )
@@
     )
   )
+  (global_label "RUN" (shape input) (at 45.72 46.99 270) (fields_autoplaced)
+    (effects (font (size 1.27 1.27)) (justify right))
+    (property "Intersheetrefs" "${INTERSHEET_REFS}" (at 45.72 53.9062 90)
+      (effects (font (size 1.27 1.27)) (justify right) hide)
+    )
+  )
   (global_label "VBUS" (shape input) (at 165.1 48.26 90) (fields_autoplaced)
     (effects (font (size 1.27 1.27)) (justify left))
@@
     )
   )
-  (global_label "RUN" (shape input) (at 45.72 46.99 180) (fields_autoplaced)
-    (effects (font (size 1.27 1.27)) (justify right))
-    (property "Intersheetrefs" "${INTERSHEET_REFS}" (at 38.8832 46.99 0)
-      (effects (font (size 1.27 1.27)) (justify right) hide)
-    )
-  )
   (global_label "USB_D+" (shape input) (at 35.56 54.61 180) (fields_autoplaced)
     (effects (font (size 1.27 1.27)) (justify right))
@@
     )
   )
+  (symbol (lib_id "Device:R_Small_US") (at 46.99 39.37 180) (unit 1)
+    (in_bom yes) (on_board yes) (dnp no) (fields_autoplaced)
+    (property "Reference" "R12" (at 49.53 38.1 0)
+      (effects (font (size 1.27 1.27)) (justify right))
+    )
+    (property "Value" "1K" (at 49.53 40.64 0)
+      (effects (font (size 1.27 1.27)) (justify right))
+    )
+    (property "Footprint" "Resistor_SMD:R_0805_2012Metric" (at 46.99 39.37 0)
+      (effects (font (size 1.27 1.27)) hide)
+    )
+    (property "Datasheet" "~" (at 46.99 39.37 0)
+      (effects (font (size 1.27 1.27)) hide)
+    )
+    (property "Link" "https://www.ozdisan.com/pasif-komponentler/direncler/smt-smd-ve-cip-direncler/0805S8F3300T5E" (at 46.99 39.37 0)
+      (effects (font (size 1.27 1.27)) hide)
+    )
+    (pin "1")
+    (pin "2")
+    (instances
+      (project "rp2040"
+        (path "/c9598c3f-0f3a-4c4d-ac85-07132829eac5"
+          (reference "R12") (unit 1)
+        )
+      )
+      (project "STM32F0_MOTOR_CONTROL_SW"
+        (path "/db7e3a52-4abf-433c-98ec-5f77753884ef/25f79f15-8146-46e0-a985-1399450076f1"
+          (reference "R?") (unit 1)
+        )
+      )
+    )
+  )
   (symbol (lib_id "power:+3.3V") (at 118.11 152.4 0) (unit 1)
     (in_bom yes) (on_board yes) (dnp no) (fields_autoplaced)
@@
     )
   )
+  (symbol (lib_id "power:+3.3V") (at 46.99 36.83 0) (unit 1)
+    (in_bom yes) (on_board yes) (dnp no) (fields_autoplaced)
+    (property "Reference" "#PWR031" (at 46.99 40.64 0)
+      (effects (font (size 1.27 1.27)) hide)
+    )
+    (property "Value" "+3.3V" (at 46.99 33.02 0)
+      (effects (font (size 1.27 1.27)))
+    )
+    (property "Footprint" "" (at 46.99 36.83 0)
+      (effects (font (size 1.27 1.27)) hide)
+    )
+    (property "Datasheet" "" (at 46.99 36.83 0)
+      (effects (font (size 1.27 1.27)) hide)
+    )
+    (pin "1")
+    (instances
+      (project "rp2040"
+        (path "/c9598c3f-0f3a-4c4d-ac85-07132829eac5"
+          (reference "#PWR031") (unit 1)
+        )
+      )
+    )
+  )
   (symbol (lib_id "power:+3.3V") (at 83.82 24.13 0) (unit 1)
     (in_bom yes) (on_board yes) (dnp no) (fields_autoplaced)
@@
     )
   )
+  (symbol (lib_id "Switch:SW_Push") (at 38.1 46.99 0) (unit 1)
+    (in_bom yes) (on_board yes) (dnp no) (fields_autoplaced)
+    (property "Reference" "SW2" (at 38.1 39.37 0)
+      (effects (font (size 1.27 1.27)))
+    )
+    (property "Value" "6x6_SMD_BUTTON" (at 38.1 41.91 0)
+      (effects (font (size 1.27 1.27)))
+    )
+    (property "Footprint" "Button_Switch_SMD:SW_SPST_CK_RS282G05A3" (at 38.1 41.91 0)
+      (effects (font (size 1.27 1.27)) hide)
+    )
+    (property "Datasheet" "~" (at 38.1 41.91 0)
+      (effects (font (size 1.27 1.27)) hide)
+    )
+    (property "Link" "ALINMAYACAK" (at 38.1 46.99 0)
+      (effects (font (size 1.27 1.27)) hide)
+    )
+    (pin "1")
+    (pin "2")
+    (instances
+      (project "rp2040"
+        (path "/c9598c3f-0f3a-4c4d-ac85-07132829eac5"
+          (reference "SW2") (unit 1)
+        )
+      )
+      (project "Cold_Room_Controller"
+        (path "/ef7b0605-ef7d-4b5f-bcde-eac45c665c82"
+          (reference "SW?") (unit 1)
+        )
+      )
+    )
+  )
   (symbol (lib_id "Device:C_Small") (at 172.72 54.61 0) (unit 1)
     (in_bom yes) (on_board yes) (dnp no)
@@
         )
       )
+    )
+  )
+  (symbol (lib_id "power:GND") (at 33.02 46.99 270) (unit 1)
+    (in_bom yes) (on_board yes) (dnp no) (fields_autoplaced)
+    (property "Reference" "#PWR030" (at 26.67 46.99 0)
+      (effects (font (size 1.27 1.27)) hide)
+    )
+    (property "Value" "GND" (at 27.94 46.99 0)
+      (effects (font (size 1.27 1.27)))
+    )
+    (property "Footprint" "" (at 33.02 46.99 0)
+      (effects (font (size 1.27 1.27)) hide)
+    )
+    (property "Datasheet" "" (at 33.02 46.99 0)
+      (effects (font (size 1.27 1.27)) hide)
+    )
+    (pin "1")
+    (instances
+      (project "rp2040"
+        (path "/c9598c3f-0f3a-4c4d-ac85-07132829eac5"
+          (reference "#PWR030") (unit 1)
+        )
+      )
